File: Hardware/Eagle/BOSS-Ion-Pump-Interface.sch (EAGLE design)
At the start: 42 parts, among them J1 MOLEX-22112022, J2 MOLEX-22112042, J3 MOLEX-22112042, J4 MOLEX-22112062, Q1 SSM3J351R, SW1 SPST-OFFBOARD, SW2 SPST-OFFBOARD, U1 ISO224ADWVR, U2 ISO224ADWVR

Commit message: Production version
Parts:
- added SW3: SPST-OFFBOARD, AUmlib:SPST-OFFBOARD
- added U$1, U$3: CON-CIRCULAR-6-OFF-BOARD, AUmlib:CON-CIRCULAR-6-OFF-BOARD
Connections:
- new net N$3: SW3.2, U$3.6
- net +15V-A: now also SW3.1
- net +5V: now also U$1.2
- net FROM-PUMP-A: now also U$3.2
- net GND: now also U$1.1
- net GND-ISO-A: now also U$3.4
- net OUTN-A: now also U$1.5
- net OUTN-B: now also U$1.4
- net OUTP-A: now also U$1.6
- net OUTP-B: now also U$1.3
- net VDD1-A: now also U$3.5
Other:
- note added: "Bulkhead connector female sockets Wire Colors 1-GRN: CASE GND 2-BLU: PUMP SIGNAL 3-NC 4-BLK: GND-ISO 5-RED: TO VDD 6-YEL: +15V"
- note added: "Bulkhead connector male pins Wire Colors 1-BLK: GND 2-RED: +5V 3-BLU: OUTB+ 4-YEL: OUTB- 5-GRN: OUTA- 6-WHT: OUTA+"
- note added: "Cable connector female sockets Wire Colors 1-BLK: GND 2-RED: +5V 3-BLU: OUTB+ 4-YEL: OUTB- 5-GRN: OUTA- 6-WHT: OUTA+"
- note added: "Cable connector male pins Wire Colors 1-NC 2-???: PUMP SIGNAL 3-NC 4-BLK: GND 5-???: +15V 6-???: +15V"
- note removed: "SIX-PINS Wire Colors 1-BLK: GND 2-RED: +5V 3-BLU: OUTB+ 4-YEL: OUTB- 5-GRN: OUTA- 6-WHT: OUTA+"
- note removed: "SIX-RECEPTACLE Wire Colors 1-GRN: CASE GND 2-BLU: PUMP SIGNAL 3-NC 4-BLK: GND-ISO 5-RED: TO VDD 6-YEL: FROM +15V"
- moved on the sheet: SW1, SW2
